Commit message: Add files via upload

File: amr_ust_description/urdf/amr_ust.xacro (robot description, xacro)
@@ -2,11 +2,13 @@
 <robot name="amr_ust" xmlns:xacro="http://www.ros.org/wiki/xacro">
 <xacro:include filename="$(find amr_ust_description)/urdf/materials.xacro" />
-<xacro:include filename="$(find amr_ust_description)/urdf/amr_ust.trans" />
+<!-- <xacro:include filename="$(find amr_ust_description)/urdf/amr_ust.trans" />  -->
 <xacro:include filename="$(find amr_ust_description)/urdf/amr_ust.gazebo" />
+<!-- <xacro:include filename="$(find amr_ust_description)/urdf/ign_material.xacro" /> -->
+<link name="base_footprint"/>
 <link name="base_link">
   <inertial>
     <origin xyz="-0.00634522824548986 -0.00013537462402944816 0.06199171397610347" rpy="0 0 0"/>
-    <mass value="${100*5.451942477570936}"/>
-    <inertia ixx="${100*0.198344}" iyy="${100*0.258519}" izz="${100*0.440587}" ixy="${100*-0.000126}" iyz="${100*3e-06}" ixz="${100*9.8e-05}"/>
+    <mass value="${1*5.451942477570936}"/>
+    <inertia ixx="${1*0.198344}" iyy="${1*0.258519}" izz="${1*0.440587}" ixy="0.0" iyz="0.0" ixz="0.0"/>
   </inertial>
   <visual>
@@ -27,6 +29,6 @@
   <inertial>
     <origin xyz="-2.639485790456586e-05 0.020563742043534228 -3.311900293296449e-05" rpy="0 0 0"/>
-    <mass value="${100*0.7547170756703072}"/>
-    <inertia ixx="${100*0.000439}" iyy="${100*0.000283}" izz="${100*0.000439}" ixy="${100*-1e-06}" iyz="${100*-1e-06}" ixz="${100*0.0}"/>
+    <mass value="${1*0.7547170756703072}"/>
+    <inertia ixx="${1*0.000439}" iyy="${1*0.000283}" izz="${1*0.000439}" ixy="0.0" iyz="0.0" ixz="0.0"/>
   </inertial>
   <visual>
@@ -47,6 +49,6 @@
   <inertial>
     <origin xyz="-2.6216982503601827e-05 -0.020564086928370973 -3.3116504283184356e-05" rpy="0 0 0"/>
-    <mass value="${100*0.7547170756701437}"/>
-    <inertia ixx="${100*0.000439}" iyy="${100*0.000283}" izz="${100*0.000439}" ixy="${100*1e-06}" iyz="${100*1e-06}" ixz="${100*0.0}"/>
+    <mass value="${1*0.7547170756701437}"/>
+    <inertia ixx="${1*0.000439}" iyy="${1*0.000283}" izz="${1*0.000439}" ixy="0.0" iyz="0.0" ixz="0.0"/>
   </inertial>
   <visual>
@@ -66,7 +68,7 @@
 <link name="wheel_hub_3_1">
   <inertial>
-    <origin xyz="-3.318509563710048e-05 0.020563634860040703 -2.6215654236647068e-05" rpy="0 0 0"/>
-    <mass value="${100*0.7547170756701448}"/>
-    <inertia ixx="${100*0.000439}" iyy="${100*0.000283}" izz="${100*0.000439}" ixy="${100*-1e-06}" iyz="${100*-1e-06}" ixz="${100*0.0}"/>
+    <origin xyz="-3.3185095637148e-05 0.020563634860040703 -2.6215654236647068e-05" rpy="0 0 0"/>
+    <mass value="${1*0.7547170756701448}"/>
+    <inertia ixx="${1*0.000439}" iyy="${1*0.000283}" izz="${1*0.000439}" ixy="0.0" iyz="0.0" ixz="0.0"/>
   </inertial>
   <visual>
@@ -87,6 +89,6 @@
   <inertial>
     <origin xyz="-2.6265710571016232e-05 -0.020564051680927398 3.311435024339754e-05" rpy="0 0 0"/>
-    <mass value="${100*0.7547170756759828}"/>
-    <inertia ixx="${100*0.000439}" iyy="${100*0.000283}" izz="${100*0.000439}" ixy="${100*1e-06}" iyz="${100*-1e-06}" ixz="${100*-0.0}"/>
+    <mass value="${1*0.7547170756759828}"/>
+    <inertia ixx="${1*0.000439}" iyy="${1*0.000283}" izz="${1*0.000439}" ixy="0.0" iyz="0.0" ixz="0.0"/>
   </inertial>
   <visual>
@@ -107,6 +109,6 @@
   <inertial>
     <origin xyz="0.017543151467361517 -0.01754284500297798 -1.0594511379302674e-11" rpy="0 0 0"/>
-    <mass value="${100*0.10437828701390915}"/>
-    <inertia ixx="${100*1.3e-05}" iyy="${100*1.3e-05}" izz="${100*2.1e-05}" ixy="${100*8e-06}" iyz="${100*-0.0}" ixz="${100*-0.0}"/>
+    <mass value="${1*0.10437828701390915}"/>
+    <inertia ixx="${1*1.3e-05}" iyy="${1*1.3e-05}" izz="${1*2.1e-05}" ixy="${1*8e-06}" iyz="${1*-0.0}" ixz="${1*-0.0}"/>
   </inertial>
   <visual>
@@ -127,6 +129,6 @@
   <inertial>
     <origin xyz="0.012404932084268683 -0.01754284500057013 -0.012404958556342202" rpy="0 0 0"/>
-    <mass value="${100*0.10437828701390915}"/>
-    <inertia ixx="${100*1.7e-05}" iyy="${100*1.3e-05}" izz="${100*1.7e-05}" ixy="${100*6e-06}" iyz="${100*-6e-06}" ixz="${100*4e-06}"/>
+    <mass value="${1*0.10437828701390915}"/>
+    <inertia ixx="${1*1.7e-05}" iyy="${1*1.3e-05}" izz="${1*1.7e-05}" ixy="${1*6e-06}" iyz="${1*-6e-06}" ixz="${1*4e-06}"/>
   </inertial>
   <visual>
@@ -147,6 +149,6 @@
   <inertial>
     <origin xyz="-3.50492340150943e-08 -0.017542844997298468 -0.017543186524848743" rpy="0 0 0"/>
-    <mass value="${100*0.10437828701390915}"/>
-    <inertia ixx="${100*2.1e-05}" iyy="${100*1.3e-05}" izz="${100*1.3e-05}" ixy="${100*0.0}" iyz="${100*-8e-06}" ixz="${100*-0.0}"/>
+    <mass value="${1*0.10437828701390915}"/>
+    <inertia ixx="${1*2.1e-05}" iyy="${1*1.3e-05}" izz="${1*1.3e-05}" ixy="${1*0.0}" iyz="${1*-8e-06}" ixz="${1*-0.0}"/>
   </inertial>
   <visual>
@@ -167,6 +169,6 @@
   <inertial>
     <origin xyz="-0.012404993591602409 -0.017542844994042683 -0.012404967140717836" rpy="0 0 0"/>
-    <mass value="${100*0.10437828701390915}"/>
-    <inertia ixx="${100*1.7e-05}" iyy="${100*1.3e-05}" izz="${100*1.7e-05}" ixy="${100*-6e-06}" iyz="${100*-6e-06}" ixz="${100*-4e-06}"/>
+    <mass value="${1*0.10437828701390915}"/>
+    <inertia ixx="${1*1.7e-05}" iyy="${1*1.3e-05}" izz="${1*1.7e-05}" ixy="${1*-6e-06}" iyz="${1*-6e-06}" ixz="${1*-4e-06}"/>
   </inertial>
   <visual>
@@ -187,6 +189,6 @@
   <inertial>
     <origin xyz="-0.017543221561155925 -0.017542844991662976 -1.0594235558269993e-11" rpy="0 0 0"/>
-    <mass value="${100*0.10437828701390915}"/>
-    <inertia ixx="${100*1.3e-05}" iyy="${100*1.3e-05}" izz="${100*2.1e-05}" ixy="${100*-8e-06}" iyz="${100*0.0}" ixz="${100*-0.0}"/>
+    <mass value="${1*0.10437828701390915}"/>
+    <inertia ixx="${1*1.3e-05}" iyy="${1*1.3e-05}" izz="${1*2.1e-05}" ixy="${1*-8e-06}" iyz="${1*0.0}" ixz="${1*-0.0}"/>
   </inertial>
   <visual>
@@ -207,6 +209,6 @@
   <inertial>
     <origin xyz="-0.012405002180593483 -0.017542844994079543 0.012404958530537124" rpy="0 0 0"/>
-    <mass value="${100*0.10437828701390915}"/>
-    <inertia ixx="${100*1.7e-05}" iyy="${100*1.3e-05}" izz="${100*1.7e-05}" ixy="${100*-6e-06}" iyz="${100*6e-06}" ixz="${100*4e-06}"/>
+    <mass value="${1*0.10437828701390915}"/>
+    <inertia ixx="${1*1.7e-05}" iyy="${1*1.3e-05}" izz="${1*1.7e-05}" ixy="${1*-6e-06}" iyz="${1*6e-06}" ixz="${1*4e-06}"/>
   </inertial>
   <visual>
@@ -227,6 +229,6 @@
   <inertial>
     <origin xyz="-3.5049233293449333e-08 -0.01754284499735176 0.017543186503658992" rpy="0 0 0"/>
-    <mass value="${100*0.10437828701390915}"/>
-    <inertia ixx="${100*2.1e-05}" iyy="${100*1.3e-05}" izz="${100*1.3e-05}" ixy="${100*-0.0}" iyz="${100*8e-06}" ixz="${100*-0.0}"/>
+    <mass value="${1*0.10437828701390915}"/>
+    <inertia ixx="${1*2.1e-05}" iyy="${1*1.3e-05}" izz="${1*1.3e-05}" ixy="${1*-0.0}" iyz="${1*8e-06}" ixz="${1*-0.0}"/>
   </inertial>
   <visual>
@@ -247,6 +249,6 @@
   <inertial>
     <origin xyz="0.01240492349527686 -0.017542845000608598 0.012404967124144517" rpy="0 0 0"/>
-    <mass value="${100*0.10437828701390915}"/>
-    <inertia ixx="${100*1.7e-05}" iyy="${100*1.3e-05}" izz="${100*1.7e-05}" ixy="${100*6e-06}" iyz="${100*6e-06}" ixz="${100*-4e-06}"/>
+    <mass value="${1*0.10437828701390915}"/>
+    <inertia ixx="${1*1.7e-05}" iyy="${1*1.3e-05}" izz="${1*1.7e-05}" ixy="${1*6e-06}" iyz="${1*6e-06}" ixz="${1*-4e-06}"/>
   </inertial>
   <visual>
@@ -267,6 +269,6 @@
   <inertial>
     <origin xyz="0.01262866495368864 0.017859997380744397 -0.01262869142546618" rpy="0 0 0"/>
-    <mass value="${100*0.1043782870139091}"/>
-    <inertia ixx="${100*1.7e-05}" iyy="${100*1.3e-05}" izz="${100*1.7e-05}" ixy="${100*-6e-06}" iyz="${100*6e-06}" ixz="${100*4e-06}"/>
+    <mass value="${1*0.1043782870139091}"/>
+    <inertia ixx="${1*1.7e-05}" iyy="${1*1.3e-05}" izz="${1*1.7e-05}" ixy="${1*-6e-06}" iyz="${1*6e-06}" ixz="${1*4e-06}"/>
   </inertial>
   <visual>
@@ -287,6 +289,6 @@
   <inertial>
     <origin xyz="0.017859557525525316 0.017859997383116 -1.0596287736142074e-11" rpy="0 0 0"/>
-    <mass value="${100*0.1043782870139091}"/>
-    <inertia ixx="${100*1.3e-05}" iyy="${100*1.3e-05}" izz="${100*2.1e-05}" ixy="${100*-8e-06}" iyz="${100*0.0}" ixz="${100*-0.0}"/>
+    <mass value="${1*0.1043782870139091}"/>
+    <inertia ixx="${1*1.3e-05}" iyy="${1*1.3e-05}" izz="${1*2.1e-05}" ixy="${1*-8e-06}" iyz="${1*0.0}" ixz="${1*-0.0}"/>
   </inertial>
   <visual>
@@ -307,6 +309,6 @@
   <inertial>
     <origin xyz="-3.504893653083485e-08 0.017859997377485448 -0.017859592582711817" rpy="0 0 0"/>
-    <mass value="${100*0.1043782870139091}"/>
-    <inertia ixx="${100*2.1e-05}" iyy="${100*1.3e-05}" izz="${100*1.3e-05}" ixy="${100*-0.0}" iyz="${100*8e-06}" ixz="${100*-0.0}"/>
+    <mass value="${1*0.1043782870139091}"/>
+    <inertia ixx="${1*2.1e-05}" iyy="${1*1.3e-05}" izz="${1*1.3e-05}" ixy="${1*-0.0}" iyz="${1*8e-06}" ixz="${1*-0.0}"/>
   </inertial>
   <visual>
@@ -327,6 +329,6 @@
   <inertial>
     <origin xyz="-0.012628726460427897 0.017859997374215952 -0.012628700009841565" rpy="0 0 0"/>
-    <mass value="${100*0.1043782870139091}"/>
-    <inertia ixx="${100*1.7e-05}" iyy="${100*1.3e-05}" izz="${100*1.7e-05}" ixy="${100*6e-06}" iyz="${100*6e-06}" ixz="${100*-4e-06}"/>
+    <mass value="${1*0.1043782870139091}"/>
+    <inertia ixx="${1*1.7e-05}" iyy="${1*1.3e-05}" izz="${1*1.7e-05}" ixy="${1*6e-06}" iyz="${1*6e-06}" ixz="${1*-4e-06}"/>
   </inertial>
   <visual>
@@ -347,6 +349,6 @@
   <inertial>
     <origin xyz="-0.017859627618709933 0.017859997371814595 -1.0596117733241428e-11" rpy="0 0 0"/>
-    <mass value="${100*0.1043782870139091}"/>
-    <inertia ixx="${100*1.3e-05}" iyy="${100*1.3e-05}" izz="${100*2.1e-05}" ixy="${100*8e-06}" iyz="${100*-0.0}" ixz="${100*-0.0}"/>
+    <mass value="${1*0.1043782870139091}"/>
+    <inertia ixx="${1*1.3e-05}" iyy="${1*1.3e-05}" izz="${1*2.1e-05}" ixy="${1*8e-06}" iyz="${1*-0.0}" ixz="${1*-0.0}"/>
   </inertial>
   <visual>
@@ -367,6 +369,6 @@
   <inertial>
     <origin xyz="-0.012628735049418499 0.017859997374192915 0.012628691399658758" rpy="0 0 0"/>
-    <mass value="${100*0.1043782870139091}"/>
-    <inertia ixx="${100*1.7e-05}" iyy="${100*1.3e-05}" izz="${100*1.7e-05}" ixy="${100*6e-06}" iyz="${100*-6e-06}" ixz="${100*4e-06}"/>
+    <mass value="${1*0.1043782870139091}"/>
+    <inertia ixx="${1*1.7e-05}" iyy="${1*1.3e-05}" izz="${1*1.7e-05}" ixy="${1*6e-06}" iyz="${1*-6e-06}" ixz="${1*4e-06}"/>
   </inertial>
   <visual>
@@ -387,6 +389,6 @@
   <inertial>
     <origin xyz="-3.5048936197767944e-08 0.017859997377449754 0.01785959256151852" rpy="0 0 0"/>
-    <mass value="${100*0.1043782870139091}"/>
-    <inertia ixx="${100*2.1e-05}" iyy="${100*1.3e-05}" izz="${100*1.3e-05}" ixy="${100*0.0}" iyz="${100*-8e-06}" ixz="${100*-0.0}"/>
+    <mass value="${1*0.1043782870139091}"/>
+    <inertia ixx="${1*2.1e-05}" iyy="${1*1.3e-05}" izz="${1*1.3e-05}" ixy="${1*0.0}" iyz="${1*-8e-06}" ixz="${1*-0.0}"/>
   </inertial>
   <visual>
@@ -407,6 +409,6 @@
   <inertial>
     <origin xyz="0.012628656364696678 0.01785999738071853 0.012628699993264443" rpy="0 0 0"/>
-    <mass value="${100*0.1043782870139091}"/>
-    <inertia ixx="${100*1.7e-05}" iyy="${100*1.3e-05}" izz="${100*1.7e-05}" ixy="${100*-6e-06}" iyz="${100*-6e-06}" ixz="${100*-4e-06}"/>
+    <mass value="${1*0.1043782870139091}"/>
+    <inertia ixx="${1*1.7e-05}" iyy="${1*1.3e-05}" izz="${1*1.7e-05}" ixy="${1*-6e-06}" iyz="${1*-6e-06}" ixz="${1*-4e-06}"/>
   </inertial>
   <visual>
@@ -427,6 +429,6 @@
   <inertial>
     <origin xyz="-0.01754322156300464 -0.01754284498951264 -1.538191796157662e-10" rpy="0 0 0"/>
-    <mass value="${100*0.10437828701391214}"/>
-    <inertia ixx="${100*1.3e-05}" iyy="${100*1.3e-05}" izz="${100*2.1e-05}" ixy="${100*-8e-06}" iyz="${100*0.0}" ixz="${100*-0.0}"/>
+    <mass value="${1*0.10437828701391214}"/>
+    <inertia ixx="${1*1.3e-05}" iyy="${1*1.3e-05}" izz="${1*2.1e-05}" ixy="${1*-8e-06}" iyz="${1*0.0}" ixz="${1*-0.0}"/>
   </inertial>
   <visual>
@@ -447,6 +449,6 @@
   <inertial>
     <origin xyz="-0.012405002182447389 -0.017542844991918383 -0.012404958694950195" rpy="0 0 0"/>
-    <mass value="${100*0.10437828701391214}"/>
-    <inertia ixx="${100*1.7e-05}" iyy="${100*1.3e-05}" izz="${100*1.7e-05}" ixy="${100*-6e-06}" iyz="${100*-6e-06}" ixz="${100*-4e-06}"/>
+    <mass value="${1*0.10437828701391214}"/>
+    <inertia ixx="${1*1.7e-05}" iyy="${1*1.3e-05}" izz="${1*1.7e-05}" ixy="${1*-6e-06}" iyz="${1*-6e-06}" ixz="${1*-4e-06}"/>
   </inertial>
   <visual>
@@ -467,6 +469,6 @@
   <inertial>
     <origin xyz="-3.5051090030435716e-08 -0.017542844995186935 -0.017543186668072128" rpy="0 0 0"/>
-    <mass value="${100*0.10437828701391214}"/>
-    <inertia ixx="${100*2.1e-05}" iyy="${100*1.3e-05}" izz="${100*1.3e-05}" ixy="${100*0.0}" iyz="${100*-8e-06}" ixz="${100*-0.0}"/>
+    <mass value="${1*0.10437828701391214}"/>
+    <inertia ixx="${1*2.1e-05}" iyy="${1*1.3e-05}" izz="${1*1.3e-05}" ixy="${1*0.0}" iyz="${1*-8e-06}" ixz="${1*-0.0}"/>
   </inertial>
   <visual>
@@ -487,6 +489,6 @@
   <inertial>
     <origin xyz="0.012404923493422093 -0.01754284499844483 -0.012404967288556236" rpy="0 0 0"/>
-    <mass value="${100*0.10437828701391214}"/>
-    <inertia ixx="${100*1.7e-05}" iyy="${100*1.3e-05}" izz="${100*1.7e-05}" ixy="${100*6e-06}" iyz="-${100*6e-06}" ixz="${100*4e-06}"/>
+    <mass value="${1*0.10437828701391214}"/>
+    <inertia ixx="${1*1.7e-05}" iyy="${1*1.3e-05}" izz="${1*1.7e-05}" ixy="${1*6e-06}" iyz="-${1*6e-06}" ixz="${1*4e-06}"/>
   </inertial>
   <visual>
@@ -507,6 +509,6 @@
   <inertial>
     <origin xyz="0.017543151465506057 -0.01754284500082315 -1.5381812143444584e-10" rpy="0 0 0"/>
-    <mass value="${100*0.10437828701391214}"/>
-    <inertia ixx="${100*1.3e-05}" iyy="${100*1.3e-05}" izz="${100*2.1e-05}" ixy="${100*8e-06}" iyz="${100*-0.0}" ixz="${100*-0.0}"/>
+    <mass value="${1*0.10437828701391214}"/>
+    <inertia ixx="${1*1.3e-05}" iyy="${1*1.3e-05}" izz="${1*2.1e-05}" ixy="${1*8e-06}" iyz="${1*-0.0}" ixz="${1*-0.0}"/>
   </inertial>
   <visual>
@@ -527,6 +529,6 @@
   <inertial>
     <origin xyz="0.01240493208241214 -0.017542844998421847 0.012404958391928143" rpy="0 0 0"/>
-    <mass value="${100*0.10437828701391214}"/>
-    <inertia ixx="${100*1.7e-05}" iyy="${100*1.3e-05}" izz="${100*1.7e-05}" ixy="${100*6e-06}" iyz="${100*6e-06}" ixz="${100*-4e-06}"/>
+    <mass value="${1*0.10437828701391214}"/>
+    <inertia ixx="${1*1.7e-05}" iyy="${1*1.3e-05}" izz="${1*1.7e-05}" ixy="${1*6e-06}" iyz="${1*6e-06}" ixz="${1*-4e-06}"/>
   </inertial>
   <visual>
@@ -547,6 +549,6 @@
   <inertial>
     <origin xyz="-0.012404993593458591 -0.017542844991894402 0.012404966976303597" rpy="0 0 0"/>
-    <mass value="${100*0.10437828701391214}"/>
-    <inertia ixx="${100*1.7e-05}" iyy="${100*1.3e-05}" izz="${100*1.7e-05}" ixy="${100*-6e-06}" iyz="${100*6e-06}" ixz="${100*4e-06}"/>
+    <mass value="${1*0.10437828701391214}"/>
+    <inertia ixx="${1*1.7e-05}" iyy="${1*1.3e-05}" izz="${1*1.7e-05}" ixy="${1*-6e-06}" iyz="${1*6e-06}" ixz="${1*4e-06}"/>
   </inertial>
   <visual>
@@ -567,6 +569,6 @@
   <inertial>
     <origin xyz="-3.505108961410208e-08 -0.01754284499515346 0.017543186360434393" rpy="0 0 0"/>
-    <mass value="${100*0.10437828701391214}"/>
-    <inertia ixx="${100*2.1e-05}" iyy="${100*1.3e-05}" izz="${100*1.3e-05}" ixy="${100*-0.0}" iyz="${100*8e-06}" ixz="${100*-0.0}"/>
+    <mass value="${1*0.10437828701391214}"/>
+    <inertia ixx="${1*2.1e-05}" iyy="${1*1.3e-05}" izz="${1*1.3e-05}" ixy="${1*-0.0}" iyz="${1*8e-06}" ixz="${1*-0.0}"/>
   </inertial>
   <visual>
@@ -587,6 +589,6 @@
   <inertial>
     <origin xyz="-0.01785962762313098 0.017859997371392433 -1.4103307410806565e-10" rpy="0 0 0"/>
-    <mass value="${100*0.10437828701391043}"/>
-    <inertia ixx="${100*1.3e-05}" iyy="${100*1.3e-05}" izz="${100*2.1e-05}" ixy="${100*8e-06}" iyz="${100*-0.0}" ixz="${100*-0.0}"/>
+    <mass value="${1*0.10437828701391043}"/>
+    <inertia ixx="${1*1.3e-05}" iyy="${1*1.3e-05}" izz="${1*2.1e-05}" ixy="${1*8e-06}" iyz="${1*-0.0}" ixz="${1*-0.0}"/>
   </inertial>
   <visual>
@@ -607,6 +609,6 @@
   <inertial>
     <origin xyz="-0.012628735053839935 0.01785999737376276 -0.012628691551287312" rpy="0 0 0"/>
-    <mass value="${100*0.10437828701391043}"/>
-    <inertia ixx="${100*1.7e-05}" iyy="${100*1.3e-05}" izz="${100*1.7e-05}" ixy="${100*6e-06}" iyz="${100*6e-06}" ixz="${100*-4e-06}"/>
+    <mass value="${1*0.10437828701391043}"/>
+    <inertia ixx="${1*1.7e-05}" iyy="${1*1.3e-05}" izz="${1*1.7e-05}" ixy="${1*6e-06}" iyz="${1*6e-06}" ixz="${1*-4e-06}"/>
   </inertial>
   <visual>
@@ -627,6 +629,6 @@
   <inertial>
     <origin xyz="-3.5053357272385455e-08 0.017859997376992898 -0.017859592713148985" rpy="0 0 0"/>
-    <mass value="${100*0.10437828701391043}"/>
-    <inertia ixx="${100*2.1e-05}" iyy="${100*1.3e-05}" izz="${100*1.3e-05}" ixy="${100*-0.0}" iyz="${100*8e-06}" ixz="${100*-0.0}"/>
+    <mass value="${1*0.10437828701391043}"/>
+    <inertia ixx="${1*2.1e-05}" iyy="${1*1.3e-05}" izz="${1*1.3e-05}" ixy="${1*-0.0}" iyz="${1*8e-06}" ixz="${1*-0.0}"/>
   </inertial>
   <visual>
@@ -647,6 +649,6 @@
   <inertial>
     <origin xyz="0.012628656360274326 0.017859997380225867 -0.012628700144894174" rpy="0 0 0"/>
-    <mass value="${100*0.10437828701391043}"/>
-    <inertia ixx="${100*1.7e-05}" iyy="${100*1.3e-05}" izz="${100*1.7e-05}" ixy="${100*-6e-06}" iyz="${100*6e-06}" ixz="${100*4e-06}"/>
+    <mass value="${1*0.10437828701391043}"/>
+    <inertia ixx="${1*1.7e-05}" iyy="${1*1.3e-05}" izz="${1*1.7e-05}" ixy="${1*-6e-06}" iyz="${1*6e-06}" ixz="${1*4e-06}"/>
   </inertial>
   <visual>
@@ -667,6 +669,6 @@
   <inertial>
     <origin xyz="0.01785955752109908 0.01785999738260663 -1.410332553866689e-10" rpy="0 0 0"/>
-    <mass value="${100*0.10437828701391043}"/>
-    <inertia ixx="${100*1.3e-05}" iyy="${100*1.3e-05}" izz="${100*2.1e-05}" ixy="${100*-8e-06}" iyz="${100*0.0}" ixz="${100*-0.0}"/>
+    <mass value="${1*0.10437828701391043}"/>
+    <inertia ixx="${1*1.3e-05}" iyy="${1*1.3e-05}" izz="${1*2.1e-05}" ixy="${1*-8e-06}" iyz="${1*0.0}" ixz="${1*-0.0}"/>
   </inertial>
   <visual>
@@ -687,6 +689,6 @@
   <inertial>
     <origin xyz="0.01262866494926565 0.017859997380236026 0.01262869127383642" rpy="0 0 0"/>
-    <mass value="${100*0.10437828701391043}"/>
-    <inertia ixx="${100*1.7e-05}" iyy="${100*1.3e-05}" izz="${100*1.7e-05}" ixy="${100*-6e-06}" iyz="${100*-6e-06}" ixz="${100*-4e-06}"/>
+    <mass value="${1*0.10437828701391043}"/>
+    <inertia ixx="${1*1.7e-05}" iyy="${1*1.3e-05}" izz="${1*1.7e-05}" ixy="${1*-6e-06}" iyz="${1*-6e-06}" ixz="${1*-4e-06}"/>
   </inertial>
   <visual>
@@ -707,6 +709,6 @@
   <inertial>
     <origin xyz="-3.505335779974139e-08 0.01785999737700683 0.017859592431082198" rpy="0 0 0"/>
-    <mass value="${100*0.10437828701391043}"/>
-    <inertia ixx="${100*2.1e-05}" iyy="${100*1.3e-05}" izz="${100*1.3e-05}" ixy="${100*0.0}" iyz="${100*-8e-06}" ixz="${100*-0.0}"/>
+    <mass value="${1*0.10437828701391043}"/>
+    <inertia ixx="${1*2.1e-05}" iyy="${1*1.3e-05}" izz="${1*1.3e-05}" ixy="${1*0.0}" iyz="${1*-8e-06}" ixz="${1*-0.0}"/>
   </inertial>
   <visual>
@@ -727,6 +729,6 @@
   <inertial>
     <origin xyz="-0.012628726464847917 0.01785999737377375 0.01262869985821194" rpy="0 0 0"/>
-    <mass value="${100*0.10437828701391043}"/>
-    <inertia ixx="${100*1.7e-05}" iyy="${100*1.3e-05}" izz="${100*1.7e-05}" ixy="${100*6e-06}" iyz="${100*-6e-06}" ixz="${100*4e-06}"/>
+    <mass value="${1*0.10437828701391043}"/>
+    <inertia ixx="${1*1.7e-05}" iyy="${1*1.3e-05}" izz="${1*1.7e-05}" ixy="${1*6e-06}" iyz="${1*-6e-06}" ixz="${1*4e-06}"/>
   </inertial>
   <visual>
@@ -747,6 +749,6 @@
   <inertial>
     <origin xyz="-0.0037135131762633944 0.00015074437785556966 -7.192465925183467e-06" rpy="0 0 0"/>
-    <mass value="${100*0.027981306586696276}"/>
-    <inertia ixx="${100*4e-06}" iyy="${100*2e-06}" izz="${2e-06}" ixy="${100*-0.0}" iyz="${100*0.0}" ixz="${100*0.0}"/>
+    <mass value="${1*0.027981306586696276}"/>
+    <inertia ixx="${1*4e-06}" iyy="${1*2e-06}" izz="${2e-06}" ixy="0.0" iyz="0.0" ixz="0.0"/>
   </inertial>
   <visual>
@@ -767,6 +769,6 @@
   <inertial>
     <origin xyz="0.017956856789517806 2.2171102201271888e-05 0.00015529819733451494" rpy="0 0 0"/>
-    <mass value="${100*0.378261563112952}"/>
-    <inertia ixx="${100*7.7e-05}" iyy="${100*9.5e-05}" izz="${100*9.3e-05}" ixy="${100*-0.0}" iyz="${100*0.0}" ixz="${100*1e-06}"/>
+    <mass value="${1*0.378261563112952}"/>
+    <inertia ixx="${1*7.7e-05}" iyy="${1*9.5e-05}" izz="${1*9.3e-05}" ixy="0.0" iyz="0.0" ixz="0.0"/>
   </inertial>
   <visual>
@@ -784,9 +786,19 @@
   </collision>
 </link>
+<link name="camera_link_depth"/>
+<link name="camera_bottom_screw_frame"/>
+<link name="camera_depth_frame"/>
+<link name="camera_depth_optical_frame"/>
+<link name="camera_color_frame"/>
+<link name="camera_color_optical_frame"/>
+<link name="camera_left_ir_frame"/>
+<link name="camera_left_ir_optical_frame"/>
+<link name="camera_right_ir_frame"/>
+<link name="camera_right_ir_optical_frame"/>
 <link name="Intel_Realsense_RPLIDAR_1">
   <inertial>
     <origin xyz="0.024168716871690317 0.00016153042204601072 0.023318927009167684" rpy="0 0 0"/>
-    <mass value="${100*1.5656994294737245}"/>
-    <inertia ixx="${100*0.000799}" iyy="${100*0.000843}" izz="${100*0.001052}" ixy="${100*-0.0}" iyz="${100*-2.9e-05}" ixz="${100*0.0}"/>
+    <mass value="${1*1.5656994294737245}"/>
+    <inertia ixx="${1*0.000799}" iyy="${1*0.000843}" izz="${1*0.001052}" ixy="0.0" iyz="0.0" ixz="0.0"/>
   </inertial>
   <visual>
@@ -804,4 +816,10 @@
   </collision>
 </link>
+<!-- BaseFootprint Joint -->
+<joint name="Fixed" type="fixed">
+  <origin xyz="0.0 0.0 0.0" rpy="0 0 0"/>
+  <parent link="base_footprint"/>
+  <child link="base_link"/>
+</joint>
 <joint name="Revolute 1" type="continuous">
   <origin xyz="0.244627 0.278967 0.032976" rpy="0 0 0"/>
@@ -1026,7 +1044,57 @@
 </joint>
 <joint name="Rigid 40" type="fixed">
-  <origin xyz="0.331142 0.000425 0.054538" rpy="0 0 0"/>
-  <parent link="base_link"/>
+  <origin xyz="0.331142 -0.000425 0.05" rpy="0 0 0"/>
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