Commit message: Add files via upload

File: amr_ust_description/urdf/amr_ust_new.urdf (robot description, URDF)
Before this commit: robot amr_ust, 42 links, 41 joints
Links:
- removed link depth_camera
- added link camera_bottom_screw_frame
- added link camera_color_frame
- added link camera_color_optical_frame
- added link camera_depth_frame
- added link camera_depth_optical_frame
- added link camera_left_ir_frame
- added link camera_left_ir_optical_frame
- added link camera_link_depth
- added link camera_right_ir_frame
- added link camera_right_ir_optical_frame
Joints:
- removed joint Rigid 43
- added joint camera_color_joint: type fixed, parent camera_depth_frame, child camera_color_frame, origin xyz=0 0 0 rpy=0 0 0
- added joint camera_color_optical_joint: type fixed, parent camera_color_frame, child camera_color_optical_frame, origin xyz=0 0 0  rpy=-1.57 0 -1.57
- added joint camera_depth_joint: type fixed, parent camera_link_depth, child camera_depth_frame, origin xyz=0 0 0 rpy=0 0 0
- added joint camera_depth_optical_joint: type fixed, parent camera_depth_frame, child camera_depth_optical_frame, origin xyz=0 0 0  rpy=-1.57 0 -1.57
- added joint camera_joint: type fixed, parent Camera_1, child camera_bottom_screw_frame, origin xyz=0 0.0 0 rpy=0 0 0
- added joint camera_left_ir_joint: type fixed, parent camera_depth_frame, child camera_left_ir_frame, origin xyz=0 0 0  rpy=0 0 0 
- added joint camera_left_ir_optical_joint: type fixed, parent camera_left_ir_frame, child camera_left_ir_optical_frame, origin xyz=0 0 0  rpy=-1.57 0 -1.57
- added joint camera_link_joint: type fixed, parent camera_bottom_screw_frame, child camera_link_depth, origin xyz=0 0.0 0.0  rpy=0 0 0
- added joint camera_right_ir_joint: type fixed, parent camera_depth_frame, child camera_right_ir_frame, origin xyz=0 -0.050 0  rpy=0 0 0
- added joint camera_right_ir_optical_joint: type fixed, parent camera_right_ir_frame, child camera_right_ir_optical_frame, origin xyz=0 0 0  rpy=-1.57 0 -1.57
- joint Rigid 40: origin xyz=0.331142 -0.1 0.054538 rpy=0 0 0 -> xyz=0.331142 -0.000425 0.1 rpy=0 0 0; parent base_link -> base_footprint
