Commit message: parameterized

File: mecanum_bot_description/urdf/amr_ust_gen.xacro (robot description, xacro)
@@ -3,7 +3,7 @@
 <xacro:include filename="$(find mecanum_bot_description)/urdf/materials.xacro" />
 <xacro:include filename="$(find mecanum_bot_description)/urdf/amr_ust.gazebo" />
-<xacro:property name="dimensions" value="mecanum_bot_params"/>
-<xacro:arg name="param_file_path" default="$(find mecanum_bot_description)/bot_config/${dimensions}.yaml" />
-<xacro:property name="bp" value="${xacro.load_yaml(param_file_path)}"/>
+<xacro:arg name="param_file_path" default="$(find mecanum_bot_description)/bot_config/mecanum_bot_params.yaml" />
+<xacro:property name="params_file" value="$(arg param_file_path)"/>
+<xacro:property name="bp" value="${xacro.load_yaml(params_file)}"/>
 <xacro:property name="mass" value="${bp['bot_mass']}"/>
 <xacro:property name="ixx" value="${bp['bot_ixx']}"/>
@@ -32,10 +32,10 @@
 <link name="base_link">
   <inertial>
-    <origin xyz="0.0 0.0 ${ground_clearance+height}" rpy="0 0 0"/>
+    <origin xyz="0.0 0.0 ${height+ground_clearance}" rpy="0 0 0"/>
     <mass value="${mass}"/>
     <inertia ixx="${ixx}" iyy="${iyy}" izz="${izz}" ixy="0.0" iyz="0.0" ixz="0.0"/>
   </inertial>
   <visual>
-    <origin xyz="0 0 0" rpy="0 0 0"/>
+    <origin xyz="0 0 ${height+ground_clearance}" rpy="0 0 0"/>
     <geometry>
       <mesh filename="file://$(find mecanum_bot_description)/meshes/base_link.stl" scale="0.001 0.001 0.001"/>
@@ -44,5 +44,5 @@
   </visual>
   <collision>
-    <origin xyz="0 0 0" rpy="0 0 0"/>
+    <origin xyz="0 0 ${height+ground_clearance}" rpy="0 0 0"/>
     <geometry>
       <mesh filename="file://$(find mecanum_bot_description)/meshes/base_link.stl" scale="0.001 0.001 0.001"/>
@@ -830,4 +830,9 @@
   </collision>
 </link>
+<joint name="fixed" type="fixed">
+  <origin xyz="0.0 0.0 0.0" rpy="0.0 0.0 0.0"/>
+  <parent link="base_footprint" />
+  <child link="base_link" />
+</joint>
 <joint name="Revolute 1" type="continuous">
   <origin xyz="0.244627 0.278967 0.032976" rpy="0 0 0"/>

Commit message: Add files via upload

File: mecanum_bot_description/urdf/amr_ust_gen.xacro (robot description, xacro)
@@ -57,5 +57,5 @@
   </inertial>
   <visual>
-    <origin xyz="-0.244627 -0.278967 -0.032976" rpy="0 0 0"/>
+    <origin xyz="${wheel_offsetX} ${wheel_offsetY} ${wheel_offsetZ}" rpy="0 0 0"/>
     <geometry>
       <mesh filename="file://$(find mecanum_bot_description)/meshes/wheel_hub_1.stl" scale="0.001 0.001 0.001"/>
@@ -64,5 +64,5 @@
   </visual>
   <collision>
-    <origin xyz="-0.244627 -0.278967 -0.032976" rpy="0 0 0"/>
+    <origin xyz="${wheel_offsetX} ${wheel_offsetY} ${wheel_offsetZ}" rpy="0 0 0"/>
     <geometry>
       <mesh filename="file://$(find mecanum_bot_description)/meshes/wheel_hub_1.stl" scale="0.001 0.001 0.001"/>

Commit message: working on parameterization

File: mecanum_bot_description/urdf/amr_ust_gen.xacro (robot description, xacro)
@@ -13,5 +13,5 @@
 <xacro:property name="width" value="${bp['chassis_width']}"/>
 <xacro:property name="height" value="${bp['chassis_height']}"/>
-<xacro:property name="ground_clearance" value="${bp['chassis_grd_clearance']}"/>
+<xacro:property name="grd_height" value="${bp['chassis_grd_height']}"/>
 <xacro:property name="wheel_mass" value="${bp['wheel_mass']}"/>
 <xacro:property name="wheel_ixx" value="${bp['wheel_inertia'][0]}"/>
@@ -26,25 +26,27 @@
 <xacro:property name="wheel_dia" value="${bp['wheel_diameter']}"/>
 <xacro:property name="wheel_thickness" value="${bp['wheel_thickness']}"/>
-<xacro:property name="wheel_offsetX" value="${bp['wheel_chassis_offsetX']}"/>
-<xacro:property name="wheel_offsetY" value="${bp['wheel_chassis_offsetY']}"/>
-<xacro:property name="wheel_offsetZ" value="${bp['wheel_chassis_offsetZ']}"/>
+<xacro:property name="wtw_l" value="${bp['wheel_to_wheel_length']}"/>
+<xacro:property name="wtw_w" value="${bp['wheel_to_wheel_width']}"/>
+<xacro:property name="wheel_offZ" value="${bp['wheel_offsetZ']}"/>
 <link name="base_footprint"/>
 <link name="base_link">
   <inertial>
-    <origin xyz="0.0 0.0 ${height+ground_clearance}" rpy="0 0 0"/>
+    <origin xyz="0.0 0.0 0.0" rpy="0 0 0"/>
     <mass value="${mass}"/>
     <inertia ixx="${ixx}" iyy="${iyy}" izz="${izz}" ixy="0.0" iyz="0.0" ixz="0.0"/>
   </inertial>
   <visual>
-    <origin xyz="0 0 ${height+ground_clearance}" rpy="0 0 0"/>
-    <geometry>
-      <mesh filename="file://$(find mecanum_bot_description)/meshes/base_link.stl" scale="0.001 0.001 0.001"/>
-    </geometry>
-    <material name="silver"/>
-  </visual>
-  <collision>
-    <origin xyz="0 0 ${height+ground_clearance}" rpy="0 0 0"/>
-    <geometry>
-      <mesh filename="file://$(find mecanum_bot_description)/meshes/base_link.stl" scale="0.001 0.001 0.001"/>
+    <origin xyz="0 0 0" rpy="0 0 0"/>
+    <geometry>
+      <!-- <mesh filename="file://$(find mecanum_bot_description)/meshes/base_link.stl" scale="0.001 0.001 0.001"/> -->
+      <box size="${length} ${width} ${height}" />
+    </geometry>
+    <material name="silver"/>
+  </visual>
+  <collision>
+    <origin xyz="0 0 0" rpy="0 0 0"/>
+    <geometry>
+      <!-- <mesh filename="file://$(find mecanum_bot_description)/meshes/base_link.stl" scale="0.001 0.001 0.001"/> -->
+      <box size="${length} ${width} ${height}"/>
     </geometry>
   </collision>
@@ -52,19 +54,21 @@
 <link name="wheel_hub_1">
   <inertial>
-    <origin xyz="-2.639485790456586e-05 0.020563742043534228 -3.311900293296449e-05" rpy="0 0 0"/>
-    <mass value="${wheel_mass}"/>
-    <inertia ixx="${wheel_ixx}" iyy="${wheel_iyy}" izz="${wheel_izz}" ixy="${wheel_ixy}" iyz="${wheel_iyz}" ixz="${wheel_ixz}"/>
-  </inertial>
-  <visual>
-    <origin xyz="${wheel_offsetX} ${wheel_offsetY} ${wheel_offsetZ}" rpy="0 0 0"/>
-    <geometry>
-      <mesh filename="file://$(find mecanum_bot_description)/meshes/wheel_hub_1.stl" scale="0.001 0.001 0.001"/>
-    </geometry>
-    <material name="silver"/>
-  </visual>
-  <collision>
-    <origin xyz="${wheel_offsetX} ${wheel_offsetY} ${wheel_offsetZ}" rpy="0 0 0"/>
-    <geometry>
-      <mesh filename="file://$(find mecanum_bot_description)/meshes/wheel_hub_1.stl" scale="0.001 0.001 0.001"/>
+    <origin xyz="0.0 0.0 0.0" rpy="0 0 0"/>
+    <mass value="${wheel_mass}"/>
+    <inertia ixx="${wheel_ixx}" iyy="${wheel_iyy}" izz="${wheel_izz}" ixy="${wheel_ixy}" iyz="${wheel_iyz}" ixz="${wheel_ixz}"/>
+  </inertial>
+  <visual>
+    <origin xyz="0 0 0" rpy="${pi/2} 0 0"/>
+    <geometry>
+      <!-- <mesh filename="file://$(find mecanum_bot_description)/meshes/wheel_hub_1.stl" scale="0.001 0.001 0.001"/> -->
+      <cylinder radius="${wheel_dia/2}"  length="${wheel_thickness}"/>
+    </geometry>
+    <material name="silver"/>
+  </visual>
+  <collision>
+    <origin xyz="0 0 0" rpy="${pi/2} 0 0"/>
+    <geometry>
+      <!-- <mesh filename="file://$(find mecanum_bot_description)/meshes/wheel_hub_1.stl" scale="0.001 0.001 0.001"/> -->
+      <cylinder radius="${wheel_dia/2}"  length="${wheel_thickness}"/>
     </geometry>
   </collision>
@@ -72,19 +76,21 @@
 <link name="wheel_hub_2_1">
   <inertial>
-    <origin xyz="-2.6216982503601827e-05 -0.020564086928370973 -3.3116504283184356e-05" rpy="0 0 0"/>
-    <mass value="${wheel_mass}"/>
-    <inertia ixx="${wheel_ixx}" iyy="${wheel_iyy}" izz="${wheel_izz}" ixy="${wheel_ixy}" iyz="${wheel_iyz}" ixz="${wheel_ixz}"/>
-  </inertial>
-  <visual>
-    <origin xyz="-0.244627 0.279033 -0.032976" rpy="0 0 0"/>
-    <geometry>
-      <mesh filename="file://$(find mecanum_bot_description)/meshes/wheel_hub_2_1.stl" scale="0.001 0.001 0.001"/>
-    </geometry>
-    <material name="silver"/>
-  </visual>
-  <collision>
-    <origin xyz="-0.244627 0.279033 -0.032976" rpy="0 0 0"/>
-    <geometry>
-      <mesh filename="file://$(find mecanum_bot_description)/meshes/wheel_hub_2_1.stl" scale="0.001 0.001 0.001"/>
+    <origin xyz="0.0 0.0 0.0" rpy="0 0 0"/>
+    <mass value="${wheel_mass}"/>
+    <inertia ixx="${wheel_ixx}" iyy="${wheel_iyy}" izz="${wheel_izz}" ixy="${wheel_ixy}" iyz="${wheel_iyz}" ixz="${wheel_ixz}"/>
+  </inertial>
+  <visual>
+    <origin xyz="0.0 0.0 0.0" rpy="${pi/2} 0 0"/>
+    <geometry>
+      <!-- <mesh filename="file://$(find mecanum_bot_description)/meshes/wheel_hub_2_1.stl" scale="0.001 0.001 0.001"/> -->
+      <cylinder radius="${wheel_dia/2}"  length="${wheel_thickness}"/>
+    </geometry>
+    <material name="silver"/>
+  </visual>
+  <collision>
+    <origin xyz="0 0 0" rpy="${pi/2} 0 0"/>
+    <geometry>
+      <!-- <mesh filename="file://$(find mecanum_bot_description)/meshes/wheel_hub_2_1.stl" scale="0.001 0.001 0.001"/> -->
+      <cylinder radius="${wheel_dia/2}"  length="${wheel_thickness}"/>
     </geometry>
   </collision>
@@ -92,19 +98,21 @@
 <link name="wheel_hub_3_1">
   <inertial>
-    <origin xyz="-3.3185095637148e-05 0.020563634860040703 -2.6215654236647068e-05" rpy="0 0 0"/>
-    <mass value="${wheel_mass}"/>
-    <inertia ixx="${wheel_ixx}" iyy="${wheel_iyy}" izz="${wheel_izz}" ixy="${wheel_ixy}" iyz="${wheel_iyz}" ixz="${wheel_ixz}"/>
-  </inertial>
-  <visual>
-    <origin xyz="0.268017 -0.278467 -0.032976" rpy="0 0 0"/>
-    <geometry>
-      <mesh filename="file://$(find mecanum_bot_description)/meshes/wheel_hub_3_1.stl" scale="0.001 0.001 0.001"/>
-    </geometry>
-    <material name="silver"/>
-  </visual>
-  <collision>
-    <origin xyz="0.268017 -0.278467 -0.032976" rpy="0 0 0"/>
-    <geometry>
-      <mesh filename="file://$(find mecanum_bot_description)/meshes/wheel_hub_3_1.stl" scale="0.001 0.001 0.001"/>
+    <origin xyz="0.0 0.0 0.0" rpy="0 0 0"/>
+    <mass value="${wheel_mass}"/>
+    <inertia ixx="${wheel_ixx}" iyy="${wheel_iyy}" izz="${wheel_izz}" ixy="${wheel_ixy}" iyz="${wheel_iyz}" ixz="${wheel_ixz}"/>
+  </inertial>
+  <visual>
+    <origin xyz="0 0 0" rpy="${pi/2} 0 0"/>
+    <geometry>
+      <!-- <mesh filename="file://$(find mecanum_bot_description)/meshes/wheel_hub_3_1.stl" scale="0.001 0.001 0.001"/> -->
+      <cylinder radius="${wheel_dia/2}"  length="${wheel_thickness}"/>
+    </geometry>
+    <material name="silver"/>
+  </visual>
+  <collision>
+    <origin xyz="0 0 0" rpy="${pi/2} 0 0"/>
+    <geometry>
+      <!-- <mesh filename="file://$(find mecanum_bot_description)/meshes/wheel_hub_3_1.stl" scale="0.001 0.001 0.001"/> -->
+      <cylinder radius="${wheel_dia/2}"  length="${wheel_thickness}"/>
     </geometry>
   </collision>
@@ -112,690 +120,33 @@
 <link name="wheel_hub_4_1">
   <inertial>
-    <origin xyz="-2.6265710571016232e-05 -0.020564051680927398 3.311435024339754e-05" rpy="0 0 0"/>
-    <mass value="${wheel_mass}"/>
-    <inertia ixx="${wheel_ixx}" iyy="${wheel_iyy}" izz="${wheel_izz}" ixy="${wheel_ixy}" iyz="${wheel_iyz}" ixz="${wheel_ixz}"/>
-  </inertial>
-  <visual>
-    <origin xyz="0.268017 0.279533 -0.032976" rpy="0 0 0"/>
-    <geometry>
-      <mesh filename="file://$(find mecanum_bot_description)/meshes/wheel_hub_4_1.stl" scale="0.001 0.001 0.001"/>
-    </geometry>
-    <material name="silver"/>
-  </visual>
-  <collision>
-    <origin xyz="0.268017 0.279533 -0.032976" rpy="0 0 0"/>
-    <geometry>
-      <mesh filename="file://$(find mecanum_bot_description)/meshes/wheel_hub_4_1.stl" scale="0.001 0.001 0.001"/>
-    </geometry>
-  </collision>
-</link>
-<link name="roller_1_1">
-  <inertial>
-    <origin xyz="0.017543151467361517 -0.01754284500297798 -1.0594511379302674e-11" rpy="0 0 0"/>
-    <mass value="${1*0.10437828701390915}"/>
-    <inertia ixx="${1*1.3e-05}" iyy="${1*1.3e-05}" izz="${1*2.1e-05}" ixy="${1*8e-06}" iyz="${1*-0.0}" ixz="${1*-0.0}"/>
-  </inertial>
-  <visual>
-    <origin xyz="-0.227018 -0.323284 -0.070476" rpy="0 0 0"/>
-    <geometry>
-      <mesh filename="file://$(find mecanum_bot_description)/meshes/roller_1_1.stl" scale="0.001 0.001 0.001"/>
-    </geometry>
-    <material name="silver"/>
-  </visual>
-  <collision>
-    <origin xyz="-0.227018 -0.323284 -0.070476" rpy="0 0 0"/>
-    <geometry>
-      <mesh filename="file://$(find mecanum_bot_description)/meshes/roller_1_1.stl" scale="0.001 0.001 0.001"/>
-    </geometry>
-  </collision>
-</link>
-<link name="roller_1_2">
-  <inertial>
-    <origin xyz="0.012404932084268683 -0.01754284500057013 -0.012404958556342202" rpy="0 0 0"/>
-    <mass value="${1*0.10437828701390915}"/>
-    <inertia ixx="${1*1.7e-05}" iyy="${1*1.3e-05}" izz="${1*1.7e-05}" ixy="${1*6e-06}" iyz="${1*-6e-06}" ixz="${1*4e-06}"/>
-  </inertial>
-  <visual>
-    <origin xyz="-0.258692 -0.323284 -0.071944" rpy="0 0 0"/>
-    <geometry>
-      <mesh filename="file://$(find mecanum_bot_description)/meshes/roller_1_2.stl" scale="0.001 0.001 0.001"/>
-    </geometry>
-    <material name="silver"/>
-  </visual>
-  <collision>
-    <origin xyz="-0.258692 -0.323284 -0.071944" rpy="0 0 0"/>
-    <geometry>
-      <mesh filename="file://$(find mecanum_bot_description)/meshes/roller_1_2.stl" scale="0.001 0.001 0.001"/>
-    </geometry>
-  </collision>
-</link>
-<link name="roller_1_3">
-  <inertial>
-    <origin xyz="-3.50492340150943e-08 -0.017542844997298468 -0.017543186524848743" rpy="0 0 0"/>
-    <mass value="${1*0.10437828701390915}"/>
-    <inertia ixx="${1*2.1e-05}" iyy="${1*1.3e-05}" izz="${1*1.3e-05}" ixy="${1*0.0}" iyz="${1*-8e-06}" ixz="${1*-0.0}"/>
-  </inertial>
-  <visual>
-    <origin xyz="-0.282127 -0.323284 -0.050585" rpy="0 0 0"/>
-    <geometry>
-      <mesh filename="file://$(find mecanum_bot_description)/meshes/roller_1_3.stl" scale="0.001 0.001 0.001"/>
-    </geometry>
-    <material name="silver"/>
-  </visual>
-  <collision>
-    <origin xyz="-0.282127 -0.323284 -0.050585" rpy="0 0 0"/>
-    <geometry>
-      <mesh filename="file://$(find mecanum_bot_description)/meshes/roller_1_3.stl" scale="0.001 0.001 0.001"/>
-    </geometry>
-  </collision>
-</link>
-<link name="roller_1_4">
-  <inertial>
-    <origin xyz="-0.012404993591602409 -0.017542844994042683 -0.012404967140717836" rpy="0 0 0"/>
-    <mass value="${1*0.10437828701390915}"/>
-    <inertia ixx="${1*1.7e-05}" iyy="${1*1.3e-05}" izz="${1*1.7e-05}" ixy="${1*-6e-06}" iyz="${1*-6e-06}" ixz="${1*-4e-06}"/>
-  </inertial>
-  <visual>
-    <origin xyz="-0.283595 -0.323284 -0.018911" rpy="0 0 0"/>
-    <geometry>
-      <mesh filename="file://$(find mecanum_bot_description)/meshes/roller_1_4.stl" scale="0.001 0.001 0.001"/>
-    </geometry>
-    <material name="silver"/>
-  </visual>
-  <collision>
-    <origin xyz="-0.283595 -0.323284 -0.018911" rpy="0 0 0"/>
-    <geometry>
-      <mesh filename="file://$(find mecanum_bot_description)/meshes/roller_1_4.stl" scale="0.001 0.001 0.001"/>
-    </geometry>
-  </collision>
-</link>
-<link name="roller_1_5">
-  <inertial>
-    <origin xyz="-0.017543221561155925 -0.017542844991662976 -1.0594235558269993e-11" rpy="0 0 0"/>
-    <mass value="${1*0.10437828701390915}"/>
-    <inertia ixx="${1*1.3e-05}" iyy="${1*1.3e-05}" izz="${1*2.1e-05}" ixy="${1*-8e-06}" iyz="${1*0.0}" ixz="${1*-0.0}"/>
-  </inertial>
-  <visual>
-    <origin xyz="-0.262236 -0.323284 0.004524" rpy="0 0 0"/>
-    <geometry>
-      <mesh filename="file://$(find mecanum_bot_description)/meshes/roller_1_5.stl" scale="0.001 0.001 0.001"/>
-    </geometry>
-    <material name="silver"/>
-  </visual>
-  <collision>
-    <origin xyz="-0.262236 -0.323284 0.004524" rpy="0 0 0"/>
-    <geometry>
-      <mesh filename="file://$(find mecanum_bot_description)/meshes/roller_1_5.stl" scale="0.001 0.001 0.001"/>
-    </geometry>
-  </collision>
-</link>
-<link name="roller_1_6">
-  <inertial>
-    <origin xyz="-0.012405002180593483 -0.017542844994079543 0.012404958530537124" rpy="0 0 0"/>
-    <mass value="${1*0.10437828701390915}"/>
-    <inertia ixx="${1*1.7e-05}" iyy="${1*1.3e-05}" izz="${1*1.7e-05}" ixy="${1*-6e-06}" iyz="${1*6e-06}" ixz="${1*4e-06}"/>
-  </inertial>
-  <visual>
-    <origin xyz="-0.230562 -0.323284 0.005992" rpy="0 0 0"/>
-    <geometry>
-      <mesh filename="file://$(find mecanum_bot_description)/meshes/roller_1_6.stl" scale="0.001 0.001 0.001"/>
-    </geometry>
-    <material name="silver"/>
-  </visual>
-  <collision>
-    <origin xyz="-0.230562 -0.323284 0.005992" rpy="0 0 0"/>
-    <geometry>
-      <mesh filename="file://$(find mecanum_bot_description)/meshes/roller_1_6.stl" scale="0.001 0.001 0.001"/>
-    </geometry>
-  </collision>
-</link>
-<link name="roller_1_7">
-  <inertial>
-    <origin xyz="-3.5049233293449333e-08 -0.01754284499735176 0.017543186503658992" rpy="0 0 0"/>
-    <mass value="${1*0.10437828701390915}"/>
-    <inertia ixx="${1*2.1e-05}" iyy="${1*1.3e-05}" izz="${1*1.3e-05}" ixy="${1*-0.0}" iyz="${1*8e-06}" ixz="${1*-0.0}"/>
-  </inertial>
-  <visual>
-    <origin xyz="-0.207127 -0.323284 -0.015367" rpy="0 0 0"/>
-    <geometry>
-      <mesh filename="file://$(find mecanum_bot_description)/meshes/roller_1_7.stl" scale="0.001 0.001 0.001"/>
-    </geometry>
-    <material name="silver"/>
-  </visual>
-  <collision>
-    <origin xyz="-0.207127 -0.323284 -0.015367" rpy="0 0 0"/>
-    <geometry>
-      <mesh filename="file://$(find mecanum_bot_description)/meshes/roller_1_7.stl" scale="0.001 0.001 0.001"/>
-    </geometry>
-  </collision>
-</link>
-<link name="roller_1_8">
-  <inertial>
-    <origin xyz="0.01240492349527686 -0.017542845000608598 0.012404967124144517" rpy="0 0 0"/>
-    <mass value="${1*0.10437828701390915}"/>
-    <inertia ixx="${1*1.7e-05}" iyy="${1*1.3e-05}" izz="${1*1.7e-05}" ixy="${1*6e-06}" iyz="${1*6e-06}" ixz="${1*-4e-06}"/>
-  </inertial>
-  <visual>
-    <origin xyz="-0.205659 -0.323284 -0.047041" rpy="0 0 0"/>
-    <geometry>
-      <mesh filename="file://$(find mecanum_bot_description)/meshes/roller_1_8.stl" scale="0.001 0.001 0.001"/>
-    </geometry>
-    <material name="silver"/>
-  </visual>
-  <collision>
-    <origin xyz="-0.205659 -0.323284 -0.047041" rpy="0 0 0"/>
-    <geometry>
-      <mesh filename="file://$(find mecanum_bot_description)/meshes/roller_1_8.stl" scale="0.001 0.001 0.001"/>
-    </geometry>
-  </collision>
-</link>
-<link name="roller_2_1">
-  <inertial>
-    <origin xyz="0.01262866495368864 0.017859997380744397 -0.01262869142546618" rpy="0 0 0"/>
-    <mass value="${1*0.1043782870139091}"/>
-    <inertia ixx="${1*1.7e-05}" iyy="${1*1.3e-05}" izz="${1*1.7e-05}" ixy="${1*-6e-06}" iyz="${1*6e-06}" ixz="${1*4e-06}"/>
-  </inertial>
-  <visual>
-    <origin xyz="-0.258692 0.323351 -0.071944" rpy="0 0 0"/>
-    <geometry>
-      <mesh filename="file://$(find mecanum_bot_description)/meshes/roller_2_1.stl" scale="0.001 0.001 0.001"/>
-    </geometry>
-    <material name="silver"/>
-  </visual>
-  <collision>
-    <origin xyz="-0.258692 0.323351 -0.071944" rpy="0 0 0"/>
-    <geometry>
-      <mesh filename="file://$(find mecanum_bot_description)/meshes/roller_2_1.stl" scale="0.001 0.001 0.001"/>
-    </geometry>
-  </collision>
-</link>
-<link name="roller_2_2">
-  <inertial>
-    <origin xyz="0.017859557525525316 0.017859997383116 -1.0596287736142074e-11" rpy="0 0 0"/>
-    <mass value="${1*0.1043782870139091}"/>
-    <inertia ixx="${1*1.3e-05}" iyy="${1*1.3e-05}" izz="${1*2.1e-05}" ixy="${1*-8e-06}" iyz="${1*0.0}" ixz="${1*-0.0}"/>
-  </inertial>
-  <visual>
-    <origin xyz="-0.227018 0.323351 -0.070476" rpy="0 0 0"/>
-    <geometry>
-      <mesh filename="file://$(find mecanum_bot_description)/meshes/roller_2_2.stl" scale="0.001 0.001 0.001"/>
-    </geometry>
-    <material name="silver"/>
-  </visual>
-  <collision>
-    <origin xyz="-0.227018 0.323351 -0.070476" rpy="0 0 0"/>
-    <geometry>
-      <mesh filename="file://$(find mecanum_bot_description)/meshes/roller_2_2.stl" scale="0.001 0.001 0.001"/>
-    </geometry>
-  </collision>
-</link>
-<link name="roller_2_3">
-  <inertial>
-    <origin xyz="-3.504893653083485e-08 0.017859997377485448 -0.017859592582711817" rpy="0 0 0"/>
-    <mass value="${1*0.1043782870139091}"/>
-    <inertia ixx="${1*2.1e-05}" iyy="${1*1.3e-05}" izz="${1*1.3e-05}" ixy="${1*-0.0}" iyz="${1*8e-06}" ixz="${1*-0.0}"/>
-  </inertial>
-  <visual>
-    <origin xyz="-0.282127 0.323351 -0.050585" rpy="0 0 0"/>
-    <geometry>
-      <mesh filename="file://$(find mecanum_bot_description)/meshes/roller_2_3.stl" scale="0.001 0.001 0.001"/>
-    </geometry>
-    <material name="silver"/>
-  </visual>
-  <collision>
-    <origin xyz="-0.282127 0.323351 -0.050585" rpy="0 0 0"/>
-    <geometry>
-      <mesh filename="file://$(find mecanum_bot_description)/meshes/roller_2_3.stl" scale="0.001 0.001 0.001"/>
-    </geometry>
-  </collision>
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