Commit message: Add files via upload

File: mecanum_bot_description/urdf/amr_ust.urdf (robot description, URDF)
Before this commit: robot amr_ust, 41 links, 39 joints
Links:
- link Camera_1: geometry collision mesh filename=file:///home/labeeb/ubot_ws/labeeb_ws/install/mecanum_bot_d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 scale=0.001 0.001 0.001; visual mesh filename=file:///home/labeeb/ubot_ws/labeeb_ws/install/mecanum_bot_d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 scale=0.001 0.001 0.001
- link Intel_Realsense_RPLIDAR_1: geometry collision mesh filename=file:///home/labeeb/ubot_ws/labeeb_ws/install/mecanum_bot_d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 scale=0.001 0.001 0.001; visual mesh filename=file:///home/labeeb/ubot_ws/labeeb_ws/install/mecanum_bot_d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 scale=0.001 0.001 0.001
- link base_link: geometry collision mesh filename=file:///home/labeeb/ubot_ws/labeeb_ws/install/mecanum_bot_d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 scale=0.001 0.001 0.001; visual mesh filename=file:///home/labeeb/ubot_ws/labeeb_ws/install/mecanum_bot_d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 scale=0.001 0.001 0.001
- link imu_link: geometry collision mesh filename=file:///home/labeeb/ubot_ws/labeeb_ws/install/mecanum_bot_d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 scale=0.001 0.001 0.001; visual mesh filename=file:///home/labeeb/ubot_ws/labeeb_ws/install/mecanum_bot_d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 scale=0.001 0.001 0.001
- link roller_1_1: geometry collision mesh filename=file:///home/labeeb/ubot_ws/labeeb_ws/install/mecanum_bot_d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 scale=0.001 0.001 0.001; visual mesh filename=file:///home/labeeb/ubot_ws/labeeb_ws/install/mecanum_bot_d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 scale=0.001 0.001 0.001
- link roller_1_2: geometry collision mesh filename=file:///home/labeeb/ubot_ws/labeeb_ws/install/mecanum_bot_d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 scale=0.001 0.001 0.001; visual mesh filename=file:///home/labeeb/ubot_ws/labeeb_ws/install/mecanum_bot_d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 scale=0.001 0.001 0.001
- link roller_1_3: geometry collision mesh filename=file:///home/labeeb/ubot_ws/labeeb_ws/install/mecanum_bot_d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 scale=0.001 0.001 0.001; visual mesh filename=file:///home/labeeb/ubot_ws/labeeb_ws/install/mecanum_bot_d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 scale=0.001 0.001 0.001
- link roller_1_4: geometry collision mesh filename=file:///home/labeeb/ubot_ws/labeeb_ws/install/mecanum_bot_d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 scale=0.001 0.001 0.001; visual mesh filename=file:///home/labeeb/ubot_ws/labeeb_ws/install/mecanum_bot_d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 scale=0.001 0.001 0.001
- link roller_1_5: geometry collision mesh filename=file:///home/labeeb/ubot_ws/labeeb_ws/install/mecanum_bot_d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 scale=0.001 0.001 0.001; visual mesh filename=file:///home/labeeb/ubot_ws/labeeb_ws/install/mecanum_bot_d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 scale=0.001 0.001 0.001
- link roller_1_6: geometry collision mesh filename=file:///home/labeeb/ubot_ws/labeeb_ws/install/mecanum_bot_d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 scale=0.001 0.001 0.001; visual mesh filename=file:///home/labeeb/ubot_ws/labeeb_ws/install/mecanum_bot_d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 scale=0.001 0.001 0.001
- link roller_1_7: geometry collision mesh filename=file:///home/labeeb/ubot_ws/labeeb_ws/install/mecanum_bot_d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 scale=0.001 0.001 0.001; visual mesh filename=file:///home/labeeb/ubot_ws/labeeb_ws/install/mecanum_bot_d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 scale=0.001 0.001 0.001
- link roller_1_8: geometry collision mesh filename=file:///home/labeeb/ubot_ws/labeeb_ws/install/mecanum_bot_d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 scale=0.001 0.001 0.001; visual mesh filename=file:///home/labeeb/ubot_ws/labeeb_ws/install/mecanum_bot_d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 scale=0.001 0.001 0.001
- link roller_2_1: geometry collision mesh filename=file:///home/labeeb/ubot_ws/labeeb_ws/install/mecanum_bot_d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 scale=0.001 0.001 0.001; visual mesh filename=file:///home/labeeb/ubot_ws/labeeb_ws/install/mecanum_bot_d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 scale=0.001 0.001 0.001
- link roller_2_2: geometry collision mesh filename=file:///home/labeeb/ubot_ws/labeeb_ws/install/mecanum_bot_d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 scale=0.001 0.001 0.001; visual mesh filename=file:///home/labeeb/ubot_ws/labeeb_ws/install/mecanum_bot_d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 scale=0.001 0.001 0.001
- link roller_2_3: geometry collision mesh filename=file:///home/labeeb/ubot_ws/labeeb_ws/install/mecanum_bot_d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 scale=0.001 0.001 0.001; visual mesh filename=file:///home/labeeb/ubot_ws/labeeb_ws/install/mecanum_bot_d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 scale=0.001 0.001 0.001
- link roller_2_4: geometry collision mesh filename=file:///home/labeeb/ubot_ws/labeeb_ws/install/mecanum_bot_d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 scale=0.001 0.001 0.001; visual mesh filename=file:///home/labeeb/ubot_ws/labeeb_ws/install/mecanum_bot_d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 scale=0.001 0.001 0.001
- link roller_2_5: geometry collision mesh filename=file:///home/labeeb/ubot_ws/labeeb_ws/install/mecanum_bot_d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 scale=0.001 0.001 0.001; visual mesh filename=file:///home/labeeb/ubot_ws/labeeb_ws/install/mecanum_bot_d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 scale=0.001 0.001 0.001
- link roller_2_6: geometry collision mesh filename=file:///home/labeeb/ubot_ws/labeeb_ws/install/mecanum_bot_d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 scale=0.001 0.001 0.001; visual mesh filename=file:///home/labeeb/ubot_ws/labeeb_ws/install/mecanum_bot_d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 scale=0.001 0.001 0.001
- link roller_2_7: geometry collision mesh filename=file:///home/labeeb/ubot_ws/labeeb_ws/install/mecanum_bot_d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 scale=0.001 0.001 0.001; visual mesh filename=file:///home/labeeb/ubot_ws/labeeb_ws/install/mecanum_bot_d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 scale=0.001 0.001 0.001
- link roller_2_8: geometry collision mesh filename=file:///home/labeeb/ubot_ws/labeeb_ws/install/mecanum_bot_d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 scale=0.001 0.001 0.001; visual mesh filename=file:///home/labeeb/ubot_ws/labeeb_ws/install/mecanum_bot_d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 scale=0.001 0.001 0.001
- link roller_3_1: geometry collision mesh filename=file:///home/labeeb/ubot_ws/labeeb_ws/install/mecanum_bot_d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 scale=0.001 0.001 0.001; visual mesh filename=file:///home/labeeb/ubot_ws/labeeb_ws/install/mecanum_bot_d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 scale=0.001 0.001 0.001
- link roller_3_2: geometry collision mesh filename=file:///home/labeeb/ubot_ws/labeeb_ws/install/mecanum_bot_d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 scale=0.001 0.001 0.001; visual mesh filename=file:///home/labeeb/ubot_ws/labeeb_ws/install/mecanum_bot_d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 scale=0.001 0.001 0.001
- link roller_3_3: geometry collision mesh filename=file:///home/labeeb/ubot_ws/labeeb_ws/install/mecanum_bot_d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 scale=0.001 0.001 0.001; visual mesh filename=file:///home/labeeb/ubot_ws/labeeb_ws/install/mecanum_bot_d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 scale=0.001 0.001 0.001
- link roller_3_4: geometry collision mesh filename=file:///home/labeeb/ubot_ws/labeeb_ws/install/mecanum_bot_d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 scale=0.001 0.001 0.001; visual mesh filename=file:///home/labeeb/ubot_ws/labeeb_ws/install/mecanum_bot_d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 scale=0.001 0.001 0.001
- link roller_3_5: geometry collision mesh filename=file:///home/labeeb/ubot_ws/labeeb_ws/install/mecanum_bot_d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 scale=0.001 0.001 0.001; visual mesh filename=file:///home/labeeb/ubot_ws/labeeb_ws/install/mecanum_bot_d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 scale=0.001 0.001 0.001
- link roller_3_6: geometry collision mesh filename=file:///home/labeeb/ubot_ws/labeeb_ws/install/mecanum_bot_d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 scale=0.001 0.001 0.001; visual mesh filename=file:///home/labeeb/ubot_ws/labeeb_ws/install/mecanum_bot_d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 scale=0.001 0.001 0.001
- link roller_3_7: geometry collision mesh filename=file:///home/labeeb/ubot_ws/labeeb_ws/install/mecanum_bot_d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 scale=0.001 0.001 0.001; visual mesh filename=file:///home/labeeb/ubot_ws/labeeb_ws/install/mecanum_bot_d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 scale=0.001 0.001 0.001
- link roller_3_8: geometry collision mesh filename=file:///home/labeeb/ubot_ws/labeeb_ws/install/mecanum_bot_d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 scale=0.001 0.001 0.001; visual mesh filename=file:///home/labeeb/ubot_ws/labeeb_ws/install/mecanum_bot_d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 scale=0.001 0.001 0.001
- link roller_4_1: geometry collision mesh filename=file:///home/labeeb/ubot_ws/labeeb_ws/install/mecanum_bot_d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 scale=0.001 0.001 0.001; visual mesh filename=file:///home/labeeb/ubot_ws/labeeb_ws/install/mecanum_bot_d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 scale=0.001 0.001 0.001
- link roller_4_2: geometry collision mesh filename=file:///home/labeeb/ubot_ws/labeeb_ws/install/mecanum_bot_d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 scale=0.001 0.001 0.001; visual mesh filename=file:///home/labeeb/ubot_ws/labeeb_ws/install/mecanum_bot_d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 scale=0.001 0.001 0.001
- link roller_4_3: geometry collision mesh filename=file:///home/labeeb/ubot_ws/labeeb_ws/install/mecanum_bot_d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 scale=0.001 0.001 0.001; visual mesh filename=file:///home/labeeb/ubot_ws/labeeb_ws/install/mecanum_bot_d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 scale=0.001 0.001 0.001
- link roller_4_4: geometry collision mesh filename=file:///home/labeeb/ubot_ws/labeeb_ws/install/mecanum_bot_d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 scale=0.001 0.001 0.001; visual mesh filename=file:///home/labeeb/ubot_ws/labeeb_ws/install/mecanum_bot_d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 scale=0.001 0.001 0.001
- link roller_4_5: geometry collision mesh filename=file:///home/labeeb/ubot_ws/labeeb_ws/install/mecanum_bot_d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 scale=0.001 0.001 0.001; visual mesh filename=file:///home/labeeb/ubot_ws/labeeb_ws/install/mecanum_bot_d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 scale=0.001 0.001 0.001
- link roller_4_6: geometry collision mesh filename=file:///home/labeeb/ubot_ws/labeeb_ws/install/mecanum_bot_d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 scale=0.001 0.001 0.001; visual mesh filename=file:///home/labeeb/ubot_ws/labeeb_ws/install/mecanum_bot_d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 scale=0.001 0.001 0.001
- link roller_4_7: geometry collision mesh filename=file:///home/labeeb/ubot_ws/labeeb_ws/install/mecanum_bot_d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 scale=0.001 0.001 0.001; visual mesh filename=file:///home/labeeb/ubot_ws/labeeb_ws/install/mecanum_bot_d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 scale=0.001 0.001 0.001
- link roller_4_8: geometry collision mesh filename=file:///home/labeeb/ubot_ws/labeeb_ws/install/mecanum_bot_d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 scale=0.001 0.001 0.001; visual mesh filename=file:///home/labeeb/ubot_ws/labeeb_ws/install/mecanum_bot_d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 scale=0.001 0.001 0.001
- link wheel_hub_1: geometry collision mesh filename=file:///home/labeeb/ubot_ws/labeeb_ws/install/mecanum_bot_d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 scale=0.001 0.001 0.001; visual mesh filename=file:///home/labeeb/ubot_ws/labeeb_ws/install/mecanum_bot_d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 scale=0.001 0.001 0.001
- link wheel_hub_2_1: geometry collision mesh filename=file:///home/labeeb/ubot_ws/labeeb_ws/install/mecanum_bot_d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 scale=0.001 0.001 0.001; visual mesh filename=file:///home/labeeb/ubot_ws/labeeb_ws/install/mecanum_bot_d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 scale=0.001 0.001 0.001
- link wheel_hub_3_1: geometry collision mesh filename=file:///home/labeeb/ubot_ws/labeeb_ws/install/mecanum_bot_d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 scale=0.001 0.001 0.001; visual mesh filename=file:///home/labeeb/ubot_ws/labeeb_ws/install/mecanum_bot_d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 scale=0.001 0.001 0.001
- link wheel_hub_4_1: geometry collision mesh filename=file:///home/labeeb/ubot_ws/labeeb_ws/install/mecanum_bot_d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 scale=0.001 0.001 0.001; visual mesh filename=file:///home/labeeb/ubot_ws/labeeb_ws/install/mecanum_bot_d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 scale=0.001 0.001 0.001
Joints:
- added joint fixed: type fixed, parent base_footprint, child base_link, origin xyz=0 0 0 rpy=0 0 0

Commit message: hardware-tested

File: mecanum_bot_description/urdf/amr_ust.urdf (robot description, URDF)
Before this commit: robot amr_ust, 41 links, 40 joints
Links:
- removed link Camera_1
- added link camera_color_frame
- added link camera_color_optical_frame
- added link camera_depth_frame
- added link camera_depth_optical_frame
- added link camera_link, mass 37.8261563112952; collision mesh filename=file:///home/inlabamr/linorobot2_ws/install/mecanum_bot_des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 scale=0.001 0.001 0.001; visual mesh filename=file:///home/inlabamr/linorobot2_ws/install/mecanum_bot_des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 scale=0.001 0.001 0.001
- link Intel_Realsense_RPLIDAR_1: geometry collision mesh filename=file:///home/inlabamr/linorobot2_ws/install/mecanum_bot_des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 scale=0.001 0.001 0.001; visual mesh filename=file:///home/inlabamr/linorobot2_ws/install/mecanum_bot_des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 scale=0.001 0.001 0.001
- link base_link: geometry collision mesh filename=file:///home/inlabamr/linorobot2_ws/install/mecanum_bot_des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 scale=0.001 0.001 0.001; visual mesh filename=file:///home/inlabamr/linorobot2_ws/install/mecanum_bot_des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 scale=0.001 0.001 0.001
- link imu_link: geometry collision mesh filename=file:///home/inlabamr/linorobot2_ws/install/mecanum_bot_des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 scale=0.001 0.001 0.001; visual mesh filename=file:///home/inlabamr/linorobot2_ws/install/mecanum_bot_des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 scale=0.001 0.001 0.001
- link roller_1_1: geometry collision mesh filename=file:///home/inlabamr/linorobot2_ws/install/mecanum_bot_des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 scale=0.001 0.001 0.001; visual mesh filename=file:///home/inlabamr/linorobot2_ws/install/mecanum_bot_des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 scale=0.001 0.001 0.001
- link roller_1_2: geometry collision mesh filename=file:///home/inlabamr/linorobot2_ws/install/mecanum_bot_des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 scale=0.001 0.001 0.001; visual mesh filename=file:///home/inlabamr/linorobot2_ws/install/mecanum_bot_des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 scale=0.001 0.001 0.001
- link roller_1_3: geometry collision mesh filename=file:///home/inlabamr/linorobot2_ws/install/mecanum_bot_des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 scale=0.001 0.001 0.001; visual mesh filename=file:///home/inlabamr/linorobot2_ws/install/mecanum_bot_des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 scale=0.001 0.001 0.001
- link roller_1_4: geometry collision mesh filename=file:///home/inlabamr/linorobot2_ws/install/mecanum_bot_des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 scale=0.001 0.001 0.001; visual mesh filename=file:///home/inlabamr/linorobot2_ws/install/mecanum_bot_des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 scale=0.001 0.001 0.001
- link roller_1_5: geometry collision mesh filename=file:///home/inlabamr/linorobot2_ws/install/mecanum_bot_des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 scale=0.001 0.001 0.001; visual mesh filename=file:///home/inlabamr/linorobot2_ws/install/mecanum_bot_des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 scale=0.001 0.001 0.001
- link roller_1_6: geometry collision mesh filename=file:///home/inlabamr/linorobot2_ws/install/mecanum_bot_des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 scale=0.001 0.001 0.001; visual mesh filename=file:///home/inlabamr/linorobot2_ws/install/mecanum_bot_des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 scale=0.001 0.001 0.001
- link roller_1_7: geometry collision mesh filename=file:///home/inlabamr/linorobot2_ws/install/mecanum_bot_des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 scale=0.001 0.001 0.001; visual mesh filename=file:///home/inlabamr/linorobot2_ws/install/mecanum_bot_des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 scale=0.001 0.001 0.001
- link roller_1_8: geometry collision mesh filename=file:///home/inlabamr/linorobot2_ws/install/mecanum_bot_des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 scale=0.001 0.001 0.001; visual mesh filename=file:///home/inlabamr/linorobot2_ws/install/mecanum_bot_des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 scale=0.001 0.001 0.001
- link roller_2_1: geometry collision mesh filename=file:///home/inlabamr/linorobot2_ws/install/mecanum_bot_des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 scale=0.001 0.001 0.001; visual mesh filename=file:///home/inlabamr/linorobot2_ws/install/mecanum_bot_des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 scale=0.001 0.001 0.001
- link roller_2_2: geometry collision mesh filename=file:///home/inlabamr/linorobot2_ws/install/mecanum_bot_des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 scale=0.001 0.001 0.001; visual mesh filename=file:///home/inlabamr/linorobot2_ws/install/mecanum_bot_des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 scale=0.001 0.001 0.001
- link roller_2_3: geometry collision mesh filename=file:///home/inlabamr/linorobot2_ws/install/mecanum_bot_des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 scale=0.001 0.001 0.001; visual mesh filename=file:///home/inlabamr/linorobot2_ws/install/mecanum_bot_des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 scale=0.001 0.001 0.001
- link roller_2_4: geometry collision mesh filename=file:///home/inlabamr/linorobot2_ws/install/mecanum_bot_des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 scale=0.001 0.001 0.001; visual mesh filename=file:///home/inlabamr/linorobot2_ws/install/mecanum_bot_des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 scale=0.001 0.001 0.001
- link roller_2_5: geometry collision mesh filename=file:///home/inlabamr/linorobot2_ws/install/mecanum_bot_des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 scale=0.001 0.001 0.001; visual mesh filename=file:///home/inlabamr/linorobot2_ws/install/mecanum_bot_des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 scale=0.001 0.001 0.001
- link roller_2_6: geometry collision mesh filename=file:///home/inlabamr/linorobot2_ws/install/mecanum_bot_des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 scale=0.001 0.001 0.001; visual mesh filename=file:///home/inlabamr/linorobot2_ws/install/mecanum_bot_des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 scale=0.001 0.001 0.001
- link roller_2_7: geometry collision mesh filename=file:///home/inlabamr/linorobot2_ws/install/mecanum_bot_des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 scale=0.001 0.001 0.001; visual mesh filename=file:///home/inlabamr/linorobot2_ws/install/mecanum_bot_des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 scale=0.001 0.001 0.001
- link roller_2_8: geometry collision mesh filename=file:///home/inlabamr/linorobot2_ws/install/mecanum_bot_des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 scale=0.001 0.001 0.001; visual mesh filename=file:///home/inlabamr/linorobot2_ws/install/mecanum_bot_des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 scale=0.001 0.001 0.001
- link roller_3_1: geometry collision mesh filename=file:///home/inlabamr/linorobot2_ws/install/mecanum_bot_des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 scale=0.001 0.001 0.001; visual mesh filename=file:///home/inlabamr/linorobot2_ws/install/mecanum_bot_des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 scale=0.001 0.001 0.001
- link roller_3_2: geometry collision mesh filename=file:///home/inlabamr/linorobot2_ws/install/mecanum_bot_des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 scale=0.001 0.001 0.001; visual mesh filename=file:///home/inlabamr/linorobot2_ws/install/mecanum_bot_des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 scale=0.001 0.001 0.001
- link roller_3_3: geometry collision mesh filename=file:///home/inlabamr/linorobot2_ws/install/mecanum_bot_des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 scale=0.001 0.001 0.001; visual mesh filename=file:///home/inlabamr/linorobot2_ws/install/mecanum_bot_des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 scale=0.001 0.001 0.001
- link roller_3_4: geometry collision mesh filename=file:///home/inlabamr/linorobot2_ws/install/mecanum_bot_des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 scale=0.001 0.001 0.001; visual mesh filename=file:///home/inlabamr/linorobot2_ws/install/mecanum_bot_des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 scale=0.001 0.001 0.001
- link roller_3_5: geometry collision mesh filename=file:///home/inlabamr/linorobot2_ws/install/mecanum_bot_des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 scale=0.001 0.001 0.001; visual mesh filename=file:///home/inlabamr/linorobot2_ws/install/mecanum_bot_des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 scale=0.001 0.001 0.001
- link roller_3_6: geometry collision mesh filename=file:///home/inlabamr/linorobot2_ws/install/mecanum_bot_des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 scale=0.001 0.001 0.001; visual mesh filename=file:///home/inlabamr/linorobot2_ws/install/mecanum_bot_des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 scale=0.001 0.001 0.001
- link roller_3_7: geometry collision mesh filename=file:///home/inlabamr/linorobot2_ws/install/mecanum_bot_des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 scale=0.001 0.001 0.001; visual mesh filename=file:///home/inlabamr/linorobot2_ws/install/mecanum_bot_des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 scale=0.001 0.001 0.001
- link roller_3_8: geometry collision mesh filename=file:///home/inlabamr/linorobot2_ws/install/mecanum_bot_des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 scale=0.001 0.001 0.001; visual mesh filename=file:///home/inlabamr/linorobot2_ws/install/mecanum_bot_des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 scale=0.001 0.001 0.001
- link roller_4_1: geometry collision mesh filename=file:///home/inlabamr/linorobot2_ws/install/mecanum_bot_des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 scale=0.001 0.001 0.001; visual mesh filename=file:///home/inlabamr/linorobot2_ws/install/mecanum_bot_des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 scale=0.001 0.001 0.001
- link roller_4_2: geometry collision mesh filename=file:///home/inlabamr/linorobot2_ws/install/mecanum_bot_des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 scale=0.001 0.001 0.001; visual mesh filename=file:///home/inlabamr/linorobot2_ws/install/mecanum_bot_des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 scale=0.001 0.001 0.001
- link roller_4_3: geometry collision mesh filename=file:///home/inlabamr/linorobot2_ws/install/mecanum_bot_des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 scale=0.001 0.001 0.001; visual mesh filename=file:///home/inlabamr/linorobot2_ws/install/mecanum_bot_des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 scale=0.001 0.001 0.001
- link roller_4_4: geometry collision mesh filename=file:///home/inlabamr/linorobot2_ws/install/mecanum_bot_des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 scale=0.001 0.001 0.001; visual mesh filename=file:///home/inlabamr/linorobot2_ws/install/mecanum_bot_des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 scale=0.001 0.001 0.001
- link roller_4_5: geometry collision mesh filename=file:///home/inlabamr/linorobot2_ws/install/mecanum_bot_des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 scale=0.001 0.001 0.001; visual mesh filename=file:///home/inlabamr/linorobot2_ws/install/mecanum_bot_des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 scale=0.001 0.001 0.001
- link roller_4_6: geometry collision mesh filename=file:///home/inlabamr/linorobot2_ws/install/mecanum_bot_des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 scale=0.001 0.001 0.001; visual mesh filename=file:///home/inlabamr/linorobot2_ws/install/mecanum_bot_des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 scale=0.001 0.001 0.001
- link roller_4_7: geometry collision mesh filename=file:///home/inlabamr/linorobot2_ws/install/mecanum_bot_des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 scale=0.001 0.001 0.001; visual mesh filename=file:///home/inlabamr/linorobot2_ws/install/mecanum_bot_des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 scale=0.001 0.001 0.001
- link roller_4_8: geometry collision mesh filename=file:///home/inlabamr/linorobot2_ws/install/mecanum_bot_des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 scale=0.001 0.001 0.001; visual mesh filename=file:///home/inlabamr/linorobot2_ws/install/mecanum_bot_des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 scale=0.001 0.001 0.001
- link wheel_hub_1: geometry collision mesh filename=file:///home/inlabamr/linorobot2_ws/install/mecanum_bot_des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 scale=0.001 0.001 0.001; visual mesh filename=file:///home/inlabamr/linorobot2_ws/install/mecanum_bot_des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 scale=0.001 0.001 0.001
- link wheel_hub_2_1: geometry collision mesh filename=file:///home/inlabamr/linorobot2_ws/install/mecanum_bot_des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 scale=0.001 0.001 0.001; visual mesh filename=file:///home/inlabamr/linorobot2_ws/install/mecanum_bot_des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 scale=0.001 0.001 0.001
- link wheel_hub_3_1: geometry collision mesh filename=file:///home/inlabamr/linorobot2_ws/install/mecanum_bot_des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 scale=0.001 0.001 0.001; visual mesh filename=file:///home/inlabamr/linorobot2_ws/install/mecanum_bot_des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 scale=0.001 0.001 0.001
- link wheel_hub_4_1: geometry collision mesh filename=file:///home/inlabamr/linorobot2_ws/install/mecanum_bot_des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 scale=0.001 0.001 0.001; visual mesh filename=file:///home/inlabamr/linorobot2_ws/install/mecanum_bot_des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 scale=0.001 0.001 0.001
Joints:
- added joint camera_color_joint: type fixed, parent camera_link, child camera_color_frame, origin xyz=0 0 0 rpy=0 0 0
- added joint camera_color_optical_joint: type fixed, parent camera_color_frame, child camera_color_optical_frame, origin xyz=0 0 0 rpy=-1.57 0 -1.57
- added joint camera_depth_joint: type fixed, parent camera_link, child camera_depth_frame, origin xyz=0 0 0 rpy=0 0 0
- added joint camera_depth_optical_joint: type fixed, parent camera_depth_frame, child camera_depth_optical_frame, origin xyz=0 0 0 rpy=-1.57 0 -1.57
- joint Rigid 40: child Camera_1 -> camera_link; origin xyz=0.331142 0.000425 0.054538 rpy=0 0 0 -> xyz=0.331142 0.0 0.054538 rpy=0 0 0
- joint Rigid 42: origin xyz=-0.024557 -0.000233 0.12 rpy=0 0 0 -> xyz=-0.0475 0.0 0.125 rpy=0 0 0
- joint fixed: origin xyz=0 0 0 rpy=0 0 0 -> xyz=0 0 0.12 rpy=0 0 0

Commit message: Oct-7-updated

File: mecanum_bot_description/urdf/amr_ust.urdf (robot description, URDF)
Before this commit: robot amr_ust, 45 links, 44 joints
Links:
- removed link Intel_Realsense_RPLIDAR_1
- added link laser, mass 156.56994294737245; collision mesh filename=file:///home/inlabamr/linorobot2_ws/install/mecanum_bot_des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 scale=0.001 0.001 0.001; visual mesh filename=file:///home/inlabamr/linorobot2_ws/install/mecanum_bot_des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 scale=0.001 0.001 0.001
Joints:
- joint Rigid 42: child Intel_Realsense_RPLIDAR_1 -> laser; origin xyz=-0.0475 0.0 0.125 rpy=0 0 0 -> xyz=0 0 0 rpy=0 0 0

Commit message: current-iteration

File: mecanum_bot_description/urdf/amr_ust.urdf (robot description, URDF)
Before this commit: robot amr_ust, 45 links, 44 joints
Links:
- removed link camera_color_frame
- removed link camera_color_optical_frame
- removed link camera_depth_frame
- removed link camera_depth_optical_frame
Joints:
- removed joint camera_color_joint
- removed joint camera_color_optical_joint
- removed joint camera_depth_joint
- removed joint camera_depth_optical_joint
- joint Rigid 42: origin xyz=0 0 0 rpy=0 0 0 -> xyz=0 0 0.208 rpy=0 0 0
